File: schematic/pods_s_charge1.kicad_sch (KiCad schematic)
At the start: 2 parts

Commit message: Owner decisions: OUT+/- rewire (CELL_NEG), XL6009 boost, server XOR
Connections:
- net GND: no longer BT1.2 (Pin_2), CHG1.2 (Pin_2)
- new net: BT1.2 (Pin_2), CHG1.2 (Pin_2)
Changed lines of the file:
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@@
     (pts
       (xy 63.5 76.2)
-      (xy 63.5 96.52)
+      (xy 63.5 91.44)
+    )
+    (stroke (width 0.1524) (type default))
+)
+  (junction (at 63.5 91.44) (diameter 0) (color 0 0 0 0)
+)
+  (wire
+    (pts
+      (xy 40.64 73.66)
+      (xy 48.26 73.66)
+    )
+    (stroke (width 0.1524) (type default))
+)
+  (wire
+    (pts
+      (xy 48.26 73.66)
+      (xy 48.26 91.44)
+    )
+    (stroke (width 0.1524) (type default))
+)
+  (junction (at 48.26 91.44) (diameter 0) (color 0 0 0 0)
+)
+  (wire
+    (pts
+      (xy 48.26 91.44)
+      (xy 63.5 91.44)
     )
     (stroke (width 0.1524) (type default))
@@
   (wire
     (pts
-      (xy 40.64 73.66)
-      (xy 48.26 73.66)
-    )
-    (stroke (width 0.1524) (type default))
-)
-  (wire
-    (pts
-      (xy 48.26 73.66)
-      (xy 48.26 96.52)
-    )
-    (stroke (width 0.1524) (type default))
-)
-  (wire
-    (pts
-      (xy 48.26 96.52)
+      (xy 55.88 96.52)
       (xy 73.66 96.52)
     )
     (stroke (width 0.1524) (type default))
 )
-  (junction (at 63.5 96.52) (diameter 0) (color 0 0 0 0)
-)
   (junction (at 68.58 96.52) (diameter 0) (color 0 0 0 0)
